File: Geiger.brd (EAGLE design)
At the start: 154.6 x 80 mm, 35 parts, among them IC1 TINY15LS, IC2 TP4056

Commit message: updates
Parts:
- added C7: (no value), resistor:C225-074X268
- added R10: 50K, resistor:R0805
- added R9: 1M, resistor:R0805
- SP1, SP2: value AL60P -> AL11P; device buzzer:AL60P -> buzzer:AL11P
- moved D1 158.4 mm to (98.7, 23.8)
- moved SP1 154.8 mm to (58.4, 27.3)
- moved ZD2 139.8 mm to (87.6, 32.4)
- moved C3 139.3 mm to (89.2, 27.3), turned to 270 degrees
- moved C2 136.3 mm to (95.6, 20.0), turned to 90 degrees
- moved R2 134.6 mm to (77.2, 36.5), turned to 90 degrees
- moved SP2 132.5 mm to (47.9, 27.3)
- moved ZD1 124.2 mm to (79.7, 32.4)
- moved D3 120.3 mm to (86.0, 23.8)
- moved D2 116.7 mm to (92.4, 23.8)
- moved R1 116.3 mm to (67.3, 24.4), turned to 90 degrees
- moved U$1 115.8 mm to (112.1, 38.7), turned to 180 degrees
- moved R3 111.1 mm to (81.6, 37.5)
- moved T1 109.8 mm to (70.5, 24.4), turned to 180 degrees
- moved C4 98.7 mm to (70.5, 31.4), turned to 180 degrees
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Connections:
- removed net N$10: ZD2.A
- removed net TR_PULSE: IC1.2, R1.1
- new net VMEASURE: IC1.2, R1.1, R10.2, R9.2
- net GND: now also C7.2, R10.1, ZD2.A
- net N$1: now also SP2.+; no longer SP2.2
- net N$8: now also C7.1
- net PULSE: now also SP1.+; no longer SP1.2
- net V+: now also SP1.-; no longer SP1.1
- net VCC: now also R9.1, SP2.-; no longer SP2.1
Routing:
- net GND: track 0.00 -> 86.0 mm
- net VCC: track 0.00 -> 47.0 mm
- net N$18: track 0.00 -> 39.0 mm
- net N$11: track 0.00 -> 30.3 mm
- net N$16: track 0.00 -> 28.7 mm
- net VMEASURE: track 0.00 -> 23.6 mm
- net N$8: track 0.00 -> 17.5 mm
- net N$5: track 0.00 -> 12.9 mm
- net N$17: track 0.00 -> 5.64 mm
- net N$6: track 0.00 -> 4.96 mm
- net N$7: track 0.00 -> 4.64 mm
- net N$21: track 0.00 -> 4.20 mm
- net N$9: track 0.00 -> 3.05 mm
- net N$2: track 0.00 -> 2.94 mm
- net N$12: track 0.00 -> 2.86 mm
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Other:
- board size 154.6 x 80 mm -> 122.2 x 47.3 mm
- board text added: "18650"

Commit message: ahoj
Parts:
- removed S1: TL36PO, switch:TL3XPO
- added JP3: PROGRAMMING, pinhead:1X04
- added R11: 1M, resistor:R0805
- added T5: (no value), transistor:SOT23-EBC
- C7: value (none) -> 100n 1KV
Connections:
- removed net N$17: C5.1, IC2.5, JP1.1, S1.2
- new net SPKR: SP1.+, T3.C
- net GND: now also JP3.4, T5.E
- net N$14: now also T5.B
- net N$22: now also JP3.3
- net N$23: now also JP3.2
- net PULSE: now also JP3.1, R11.2, T5.C; no longer SP1.+, T3.C
- net VCC: now also C5.1, IC2.5, JP1.1, R11.1; no longer S1.1
Routing:
- net N$17: track 5.64 -> 0.00 mm
- net VCC: track 47.0 -> 52.6 mm
Changed lines of the file:
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@@
 <?xml version="1.0" encoding="utf-8"?>
 <!DOCTYPE eagle SYSTEM "eagle.dtd">
-<eagle version="7.7.0">
+<eagle version="7.6.0">
 <drawing>
 <settings>
@@
 <element name="R6" library="resistor" package="R1206" value="0R39" x="10.795" y="28.8925" rot="R180"/>
 <element name="R7" library="resistor" package="R0805" value="3K" x="17.4625" y="29.845" rot="R270"/>
-<element name="S1" library="switch" package="TL3XPO" value="TL36PO" x="-50.8" y="6.35"/>
 <element name="T1" library="transistor" package="SOT23-EBC" value="" x="70.485" y="24.4475" rot="R180"/>
 <element name="T2" library="transistor" package="SOT23-BCE" value="" x="-39.37" y="57.15"/>
@@
 <element name="R9" library="resistor" package="R0805" value="1M" x="-95.25" y="-33.02"/>
 <element name="R10" library="resistor" package="R0805" value="50K" x="-95.25" y="-39.37"/>
-<element name="C7" library="resistor" package="C225-074X268" value="" x="87.9475" y="27.305"/>
+<element name="C7" library="resistor" package="C225-074X268" value="100n 1KV" x="87.9475" y="27.305"/>
 <element name="SP2" library="buzzer" package="AL11P" value="AL11P" x="47.9425" y="27.305">
 <attribute name="OC_NEWARK" value="unknown" x="47.9425" y="27.305" size="1.778" layer="27" display="off"/>
@@
 <attribute name="MF" value="" x="58.42" y="27.305" size="1.778" layer="27" display="off"/>
 </element>
+<element name="JP3" library="pinhead" package="1X04" value="PROGRAMMING" x="-91.44" y="-46.0375"/>
+<element name="T5" library="transistor" package="SOT23-EBC" value="" x="-94.615" y="-53.34"/>
+<element name="R11" library="resistor" package="R0805" value="1M" x="-95.25" y="-58.42"/>
 </elements>
 <signals>
@@
 <contactref element="T2" pad="E"/>
 <contactref element="S2" pad="3"/>
-<contactref element="S1" pad="1"/>
 <contactref element="R9" pad="1"/>
 <contactref element="SP2" pad="-"/>
@@
 <wire x1="66.675" y1="36.195" x2="67.9425" y2="36.195" width="0.8128" layer="1"/>
 <wire x1="67.9425" y1="36.195" x2="67.945" y2="36.1925" width="0.8128" layer="1"/>
+<contactref element="IC2" pad="5"/>
+<contactref element="C5" pad="1"/>
+<contactref element="JP1" pad="1"/>
+<wire x1="25.2925" y1="26.035" x2="27.305" y2="26.035" width="0.6096" layer="1"/>
+<wire x1="27.305" y1="26.035" x2="27.305" y2="26.0325" width="0.6096" layer="1"/>
+<wire x1="27.305" y1="26.0325" x2="30.4825" y2="26.0325" width="0.6096" layer="1"/>
+<wire x1="30.4825" y1="26.0325" x2="30.7975" y2="25.7175" width="0.6096" layer="1"/>
+<contactref element="R11" pad="1"/>
+<wire x1="-96.2" y1="-33.02" x2="-96.2" y2="-58.42" width="0" layer="19" extent="1-1"/>
 <wire x1="-63.5" y1="6.35" x2="-96.2" y2="-33.02" width="0" layer="19" extent="1-1"/>
-<wire x1="-53.34" y1="6.35" x2="-63.5" y2="6.35" width="0" layer="19" extent="1-1"/>
-<wire x1="-39.8" y1="52.07" x2="-53.34" y2="6.35" width="0" layer="19" extent="1-1"/>
+<wire x1="-39.8" y1="52.07" x2="-63.5" y2="6.35" width="0" layer="19" extent="1-1"/>
 <wire x1="-39.37" y1="58.25" x2="-39.8" y2="52.07" width="0" layer="19" extent="1-1"/>
-<wire x1="45.9105" y1="27.305" x2="-39.8" y2="52.07" width="0" layer="19" extent="1-1"/>
+<wire x1="25.2925" y1="26.035" x2="-39.8" y2="52.07" width="0" layer="19" extent="1-1"/>
+<wire x1="45.9105" y1="27.305" x2="30.7975" y2="25.7175" width="0" layer="19" extent="1-1"/>
 <wire x1="59.6875" y1="40.6425" x2="45.9105" y2="27.305" width="0" layer="19" extent="1-1"/>
 </signal>
@@
 <wire x1="55.88" y1="36.195" x2="54.9585" y2="36.195" width="0.8128" layer="1"/>
 <wire x1="54.9585" y1="36.195" x2="54.9485" y2="36.205" width="0.8128" layer="1"/>
+<contactref element="JP3" pad="4"/>
+<contactref element="T5" pad="E"/>
+<wire x1="-87.63" y1="-46.0375" x2="-95.565" y2="-54.44" width="0" layer="19" extent="1-1"/>
+<wire x1="-96.2" y1="-39.37" x2="-87.63" y2="-46.0375" width="0" layer="19" extent="1-1"/>
 <wire x1="-94.93" y1="-22.69" x2="-96.2" y2="-39.37" width="0" layer="19" extent="1-1"/>
 <wire x1="-68.58" y1="6.35" x2="-94.93" y2="-22.69" width="0" layer="19" extent="1-1"/>
@@
 <contactref element="R5" pad="1"/>
 <contactref element="T3" pad="B"/>
-<wire x1="-53.02" y1="45.72" x2="-43.5" y2="56.05" width="0" layer="19" extent="1-1"/>
+<contactref element="T5" pad="B"/>
+<wire x1="-53.02" y1="45.72" x2="-93.665" y2="-54.44" width="0" layer="19" extent="1-1"/>
+<wire x1="-43.5" y1="56.05" x2="-53.02" y2="45.72" width="0" layer="19" extent="1-1"/>
 </signal>
 <signal name="PULSE">
 <contactref element="IC1" pad="7"/>
-<contactref element="T3" pad="C"/>
-<contactref element="SP1" pad="+"/>
-<wire x1="60.452" y1="27.305" x2="61.2565" y2="38.735" width="0" layer="19" extent="1-1"/>
-<wire x1="-44.45" y1="58.25" x2="61.2565" y2="38.735" width="0" layer="19" extent="1-1"/>
+<contactref element="JP3" pad="1"/>
+<contactref element="R11" pad="2"/>
+<contactref element="T5" pad="C"/>
+<wire x1="-94.615" y1="-52.24" x2="-94.3" y2="-58.42" width="0" layer="19" extent="1-1"/>
+<wire x1="-95.25" y1="-46.0375" x2="-94.615" y2="-52.24" width="0" layer="19" extent="1-1"/>
+<wire x1="61.2565" y1="38.735" x2="-95.25" y2="-46.0375" width="0" layer="19" extent="1-1"/>
 </signal>
 <signal name="N$13">
@@
 <wire x1="12.217" y1="28.8925" x2="15.5575" y2="28.8925" width="0.6096" layer="1"/>
 </signal>
-<signal name="N$17">
-<contactref element="IC2" pad="5"/>
-<contactref element="C5" pad="1"/>
-<contactref element="JP1" pad="1"/>
-<contactref element="S1" pad="2"/>
-<wire x1="25.2925" y1="26.035" x2="27.305" y2="26.035" width="0.6096" layer="1"/>
-<wire x1="27.305" y1="26.035" x2="27.305" y2="26.0325" width="0.6096" layer="1"/>
-<wire x1="27.305" y1="26.0325" x2="30.4825" y2="26.0325" width="0.6096" layer="1"/>
-<wire x1="30.4825" y1="26.0325" x2="30.7975" y2="25.7175" width="0.6096" layer="1"/>
-<wire x1="-50.8" y1="6.35" x2="25.2925" y2="26.035" width="0" layer="19" extent="1-1"/>
-</signal>
 <signal name="N$19">
 <contactref element="IC2" pad="2"/>
@@
 <contactref element="IC1" pad="5"/>
 <contactref element="JP2" pad="1"/>
-<wire x1="-38.1" y1="27.94" x2="61.2565" y2="36.195" width="0" layer="19" extent="1-1"/>
+<contactref element="JP3" pad="3"/>
+<wire x1="-38.1" y1="27.94" x2="-90.17" y2="-46.0375" width="0" layer="19" extent="1-1"/>
+<wire x1="61.2565" y1="36.195" x2="-38.1" y2="27.94" width="0" layer="19" extent="1-1"/>
 </signal>
 <signal name="N$23">
 <contactref element="JP2" pad="2"/>
 <contactref element="IC1" pad="6"/>
-<wire x1="-35.56" y1="27.94" x2="61.2565" y2="37.465" width="0" layer="19" extent="1-1"/>
+<contactref element="JP3" pad="2"/>
+<wire x1="-35.56" y1="27.94" x2="-92.71" y2="-46.0375" width="0" layer="19" extent="1-1"/>
+<wire x1="61.2565" y1="37.465" x2="-35.56" y2="27.94" width="0" layer="19" extent="1-1"/>
 </signal>
 <signal name="N$18">
@@
 <wire x1="111.76" y1="39.0525" x2="112.0775" y2="38.735" width="0.8128" layer="1"/>
 </signal>
+<signal name="SPKR">
+<contactref element="T3" pad="C"/>
+<contactref element="SP1" pad="+"/>
+<wire x1="-44.45" y1="58.25" x2="60.452" y2="27.305" width="0" layer="19" extent="1-1"/>
+</signal>
 </signals>

Commit message: dalsi
Parts:
- removed C7: 100n 1KV, resistor:C225-074X268
- removed R6: 0R39, resistor:R1206
- removed T2: (no value), transistor:SOT23-BCE
- added C8: 100n, resistor:C0805
- added C9: 100n 500V, resistor:C150-054X183
- added JP4: RESET, pinhead:1X01
- added R12: 0R39, resistor:R2512
- T1, T3, T4, T5: device transistor:SOT23-EBC -> transistor:SOT23-BEC
- moved T5 224.4 mm to (129.5, -42.5)
- moved R5 174.2 mm to (111.1, -15.2), turned to 90 degrees
- moved T3 172.7 mm to (110.2, -19.7), turned to 180 degrees
- moved D4 170.7 mm to (121.0, -9.84), turned to 270 degrees
- moved R1 142.8 mm to (-62.2, -35.6), turned to 180 degrees
- moved IC1 135.5 mm to (-55.2, -36.2)
- moved C1 133.4 mm to (-52.1, -32.1)
- moved SP2 120.0 mm to (-62.9, -18.7)
- moved R2 84.8 mm to (145.1, -14.3), turned to 180 degrees
- moved ZD1 82.2 mm to (143.8, -19.1), turned to 180 degrees
- moved R3 78.8 mm to (143.8, -10.8), turned to 90 degrees
- moved TRANSFORMER 77.9 mm to (141.3, -32.1)
- moved D2 77.3 mm to (140.7, -36.5), turned to 270 degrees
- moved D3 76.8 mm to (140.7, -30.2), turned to 270 degrees
- moved C2 76.6 mm to (145.1, -38.4), turned to 180 degrees
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Connections:
- removed net N$21: R6.2, U1.VBUS1
- new net GNDUSB: R12.2, U1.VBUS1
- new net N$10: R11.1, R5.2, T1.C
- net ALARM: now also C8.1, R10.2, R9.2
- net GND: now also C8.2, C9.2; no longer C7.2, T1.E
- net N$12: now also T1.B; no longer T2.B
- net N$13: now also IC1.1, JP4.1; no longer R5.2, T2.C
- net N$14: no longer T5.B
- net N$16: now also R12.1; no longer R6.1
- net N$18: now also T5.C; no longer T1.C
- net N$4: now also T5.B; no longer T1.B
- net N$8: now also C9.1; no longer C7.1
- net PULSE: no longer T5.C
- net VCC: now also T1.E; no longer R11.1, T2.E
- net VMEASURE: no longer R10.2, R9.2
Routing:
- net GND: track 86.0 -> 139.9 mm
- net N$11: track 30.3 -> 0.00 mm
- net VCC: track 52.6 -> 25.5 mm
- net N$18: track 39.0 -> 16.9 mm
- net VMEASURE: track 23.6 -> 2.91 mm
- net N$23: track 0.00 -> 19.8 mm
- net N$22: track 0.00 -> 19.2 mm
- net ALARM: track 0.00 -> 17.5 mm
- net PULSE: track 0.00 -> 15.1 mm
- net N$12: track 2.86 -> 12.2 mm
- net N$5: track 12.9 -> 21.9 mm
- net N$10: track 0.00 -> 6.34 mm
- net N$3: track 0.00 -> 6.32 mm
- net N$1: track 0.00 -> 5.55 mm
- net N$21: track 4.20 -> 0.00 mm
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Other:
- board size 122.2 x 47.3 mm -> 136.8 x 47.6 mm

Commit message: co asi
Parts:
- removed IC2: TP4056, TP4056:SOP-8
- removed JP1: BATTERY, pinhead:1X02
- removed R12: 0R39, resistor:R2512
- removed U1: (no value), MicroUSB:USB-MICRO-SMD
- added IC3: TP4056, Geiger:SOP-8
- added R6: 1M, resistor:0207/7
- added S1: TL36PO, switch:TL3XPO
- added U2: USB, Geiger:USB-MICRO-SMD
- R2: value 1M -> 0R39; device resistor:R0805 -> resistor:R1206
- R3: value 5M1 -> 4M3
- T1: value (none) -> BC807
- T3, T4, T5: value (none) -> 3904
- moved R2 141.4 mm to (10.2, 27.9)
- moved JP4 135.9 mm to (58.4, 30.5)
- moved R1 135.6 mm to (57.8, 27.6)
- moved C8 135.5 mm to (66.0, 35.9)
- moved R10 135.5 mm to (66.0, 33.3)
- moved C1 135.5 mm to (67.9, 30.8)
- moved IC1 135.5 mm to (64.8, 26.7)
- moved R8 135.5 mm to (61.6, 35.9)
- moved R9 135.5 mm to (61.6, 33.3)
- moved JP3 133.3 mm to (75.6, 27.6)
- moved R11 133.3 mm to (75.6, 35.6)
- moved JP2 131.6 mm to (81.0, 27.6)
- moved T4 121.4 mm to (52.1, 34.3), turned to 90 degrees
- moved SP2 118.1 mm to (45.7, 27.6), turned to 180 degrees
- moved S2 81.9 mm to (34.6, 24.1), turned to 0 degrees
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Connections:
- net N$6 renamed 200V2
- net N$7 renamed 400V3
- net N$9 renamed 200V
- removed net GNDUSB: R12.2, U1.VBUS1
- removed net N$5: C4.1, R2.2, R3.1
- removed net N$8: C9.1, D3.C, R2.1, ZD1.C
- new net 400V: C9.1, D3.C, R6.1, ZD1.C
- new net 400V2: C4.1, R3.1, R6.2
- new net N$15: S1.2, S1.3
- new net VCCUSB: R2.2, U2.VBUS1
- net GND: now also IC3.1, IC3.3, IC3.P$1, JP2.2, U2.GND1; no longer IC2.1, IC2.3, JP1.2, JP2.4, U1.GND1
- net N$16: now also IC3.4, IC3.8, R2.1; no longer IC2.4, IC2.8, R12.1
- net N$19: now also IC3.2; no longer IC2.2
- net N$22: now also JP2.3; no longer JP2.1
- net N$23: now also JP2.4; no longer JP2.2
- net V+: now also JP2.1; no longer JP2.3
- net VCC: now also IC3.5, S1.1; no longer IC2.5, JP1.1
Routing:
- net VCC: track 25.5 -> 171.5 mm, vias 0 -> 2
- net V+: track 0.00 -> 125.8 mm
- net GND: track 139.9 -> 243.4 mm
- net N$4: track 2.06 -> 62.0 mm, vias 0 -> 2
- net A: track 0.00 -> 46.1 mm
- net N$10: track 6.34 -> 44.9 mm
- net N$18: track 16.9 -> 41.6 mm
- net N$5: track 21.9 -> 0.00 mm
- net N$8: track 21.5 -> 0.00 mm
- net N$11: track 0.00 -> 17.3 mm
- net 400V: track 0.00 -> 12.0 mm
- net 400V2: track 0.00 -> 10.6 mm
- net N$13: track 0.00 -> 4.92 mm
- net N$1: track 5.55 -> 10.2 mm
- net VCCUSB: track 0.00 -> 4.25 mm
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- added copper zone on layer 1, net GND
- added copper zone on layer 1, net VCCUSB
Other:
- board size 136.8 x 47.6 mm -> 137.1 x 47.9 mm
- board text added: "hertdani"

Commit message: dalsi
Parts:
- removed D1, D2, D3: BAV21W, diode:SOD123
- added D5, D6, D7: EGL1G, diode:SOD80C
- added R12, R13, R14: 1M, resistor:R0805
- R3: value 4M3 -> 1M
- R6: device resistor:0207/7 -> resistor:R0805
- moved R5 32.6 mm to (81.6, 34.6), turned to 180 degrees
- moved T3 29.1 mm to (86.7, 30.5)
- moved SP1 29.1 mm to (90.5, 27.6), turned to 90 degrees
- moved C3 19.1 mm to (110.8, 13.3)
- moved ZD1 18.6 mm to (112.7, 20.3)
- moved C9 17.2 mm to (108.9, 23.5)
- moved ZD2 15.9 mm to (105.1, 20.3)
- moved T5 13.5 mm to (92.1, 17.8), turned to 180 degrees
- moved C4 10.9 mm to (100.6, 28.3)
- moved R6 9.38 mm to (99.1, 36.5), turned to 270 degrees
- moved TRANSFORMER 9.26 mm to (83.8, 16.5)
- moved C2 8.64 mm to (104.8, 3.49), turned to 0 degrees
- moved R3 6.79 mm to (103.2, 31.8), turned to 270 degrees
- moved SP2 2.22 mm to (43.5, 27.6), turned to 90 degrees
- moved T1 2.03 mm to (82.9, 38.1)
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Connections:
- net VMEASURE renamed OSC
- removed net N$11: R3.2, U$1.P$1
- new net N$6: R3.1, R6.2
- new net N$7: R13.2, R6.1
- new net N$8: R14.1, U$1.P$1
- new net N$9: R13.1, R14.2
- net 200V2: now also D5.C, D6.A; no longer D1.C, D2.A
- net 400V: now also D7.C, R12.1; no longer D3.C, R6.1
- net 400V2: now also R12.2, R3.2; no longer R3.1, R6.2
- net 400V3: now also D6.C, D7.A; no longer D2.C, D3.A
- net GND: now also D5.A; no longer D1.A
Routing:
- net V+: track 125.8 -> 60.6 mm
- net N$10: track 44.9 -> 10.2 mm
- net N$18: track 41.6 -> 18.5 mm
- net N$11: track 17.3 -> 0.00 mm
- net N$8: track 0.00 -> 9.68 mm
- net N$12: track 9.28 -> 17.8 mm
- net N$4: track 62.0 -> 53.7 mm
- net VCC: track 171.5 -> 178.2 mm
- net 200V2: track 6.94 -> 12.4 mm
- net 400V2: track 10.6 -> 15.8 mm
- net N$6: track 0.00 -> 5.18 mm
- net GND: track 243.4 -> 238.6 mm
- net N$14: track 2.62 -> 5.51 mm
- net 400V3: track 5.22 -> 7.94 mm
- net N$9: track 0.00 -> 2.67 mm
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Other:
- board size 137.1 x 47.9 mm -> 120.3 x 47.6 mm
- board text added: "Geiger Counter"

Commit message: fsldi
Parts:
- moved D7 1.71 mm to (115.6, 15.9)
Routing:
- net 400V3: track 7.94 -> 5.67 mm
