File: Geiger.brd (EAGLE design)
At the start: 120.3 x 47.6 mm, 44 parts, among them IC1 TINY15LS, IC3 TP4056, T1 BC807, T3 3904, T4 3904, T5 3904, U2 USB

Commit message: Minor updates
Routing:
- net GND: vias 0 -> 2
Changed lines of the file:
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@@
 <wire x1="106.9975" y1="10.255" x2="106.9975" y2="12.3825" width="0.8128" layer="1"/>
 <wire x1="106.9975" y1="12.3825" x2="107.95" y2="13.335" width="0.8128" layer="1"/>
+<via x="21.9075" y="27.94" extent="1-16" drill="0.8"/>
+<via x="21.9075" y="26.035" extent="1-16" drill="0.8"/>
 </signal>
 <signal name="N$4">
@@
 <wire x1="100.015" y1="42.8625" x2="99.06" y2="42.06625" width="0.8128" layer="1"/>
 </signal>
-<signal name="N$5">
-<via x="21.9075" y="26.035" extent="1-16" drill="0.8"/>
-</signal>
-<signal name="N$11">
-<via x="21.9075" y="27.94" extent="1-16" drill="0.8"/>
-</signal>
 </signals>

Commit message: update
Routing:
- net N$5: track 0.00 -> 335.9 mm
Changed lines of the file:
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@@
 <setting verticaltext="up"/>
 </settings>
-<grid distance="0.0125" unitdist="inch" unit="inch" style="lines" multiple="1" display="yes" altdistance="0.025" altunitdist="inch" altunit="inch"/>
+<grid distance="0.0125" unitdist="inch" unit="mm" style="lines" multiple="1" display="yes" altdistance="0.025" altunitdist="inch" altunit="inch"/>
 <layers>
 <layer number="1" name="Top" color="4" fill="1" visible="yes" active="yes"/>
@@
 <layer number="17" name="Pads" color="2" fill="1" visible="yes" active="yes"/>
 <layer number="18" name="Vias" color="2" fill="1" visible="yes" active="yes"/>
-<layer number="19" name="Unrouted" color="6" fill="1" visible="yes" active="yes"/>
-<layer number="20" name="Dimension" color="15" fill="1" visible="yes" active="yes"/>
-<layer number="21" name="tPlace" color="7" fill="1" visible="yes" active="yes"/>
-<layer number="22" name="bPlace" color="7" fill="1" visible="yes" active="yes"/>
-<layer number="23" name="tOrigins" color="15" fill="1" visible="yes" active="yes"/>
-<layer number="24" name="bOrigins" color="15" fill="1" visible="yes" active="yes"/>
-<layer number="25" name="tNames" color="7" fill="1" visible="yes" active="yes"/>
+<layer number="19" name="Unrouted" color="6" fill="1" visible="no" active="yes"/>
+<layer number="20" name="Dimension" color="15" fill="1" visible="no" active="yes"/>
+<layer number="21" name="tPlace" color="7" fill="1" visible="no" active="yes"/>
+<layer number="22" name="bPlace" color="7" fill="1" visible="no" active="yes"/>
+<layer number="23" name="tOrigins" color="15" fill="1" visible="no" active="yes"/>
+<layer number="24" name="bOrigins" color="15" fill="1" visible="no" active="yes"/>
+<layer number="25" name="tNames" color="7" fill="1" visible="no" active="yes"/>
 <layer number="26" name="bNames" color="7" fill="1" visible="no" active="yes"/>
 <layer number="27" name="tValues" color="7" fill="1" visible="no" active="yes"/>
@@
 <layer number="37" name="tTest" color="7" fill="1" visible="no" active="yes"/>
 <layer number="38" name="bTest" color="7" fill="1" visible="no" active="yes"/>
-<layer number="39" name="tKeepout" color="4" fill="11" visible="yes" active="yes"/>
+<layer number="39" name="tKeepout" color="4" fill="11" visible="no" active="yes"/>
 <layer number="40" name="bKeepout" color="1" fill="11" visible="no" active="yes"/>
-<layer number="41" name="tRestrict" color="4" fill="10" visible="yes" active="yes"/>
+<layer number="41" name="tRestrict" color="4" fill="10" visible="no" active="yes"/>
 <layer number="42" name="bRestrict" color="1" fill="10" visible="no" active="yes"/>
 <layer number="43" name="vRestrict" color="2" fill="10" visible="no" active="yes"/>
@@
 <layer number="49" name="Reference" color="7" fill="1" visible="no" active="yes"/>
 <layer number="50" name="dxf" color="7" fill="1" visible="no" active="no"/>
-<layer number="51" name="tDocu" color="7" fill="1" visible="yes" active="yes"/>
+<layer number="51" name="tDocu" color="7" fill="1" visible="no" active="yes"/>
 <layer number="52" name="bDocu" color="7" fill="1" visible="no" active="yes"/>
 <layer number="53" name="tGND_GNDA" color="7" fill="1" visible="no" active="no"/>
@@
 <layer number="114" name="Badge_Outline" color="7" fill="1" visible="no" active="yes"/>
 <layer number="115" name="ReferenceISLANDS" color="7" fill="1" visible="no" active="yes"/>
-<layer number="116" name="Patch_BOT" color="9" fill="4" visible="no" active="yes"/>
+<layer number="116" name="centerDrill" color="9" fill="4" visible="yes" active="yes"/>
 <layer number="118" name="Rect_Pads" color="7" fill="1" visible="no" active="yes"/>
 <layer number="121" name="_tsilk" color="7" fill="1" visible="no" active="yes"/>
@@
 <text x="18.0975" y="42.8625" size="3.556" layer="1" font="vector" ratio="16">hertdani</text>
 <text x="45.4025" y="42.8625" size="3.556" layer="1" font="vector" ratio="16">Geiger Counter</text>
+<circle x="103.188" y="28.258" radius="0.424" width="0.05" layer="116"/>
+<circle x="98.108" y="28.258" radius="0.424" width="0.05" layer="116"/>
+<circle x="116.396" y="23.495" radius="0.425" width="0.05" layer="116"/>
+<circle x="101.41" y="23.495" radius="0.425" width="0.05" layer="116"/>
+<circle x="82.233" y="23.812" radius="0.424" width="0.05" layer="116"/>
+<circle x="82.233" y="26.353" radius="0.424" width="0.05" layer="116"/>
+<circle x="82.233" y="28.893" radius="0.424" width="0.05" layer="116"/>
+<circle x="82.233" y="31.433" radius="0.424" width="0.05" layer="116"/>
+<circle x="76.835" y="31.433" radius="0.425" width="0.05" layer="116"/>
+<circle x="76.835" y="28.893" radius="0.425" width="0.05" layer="116"/>
+<circle x="76.835" y="26.353" radius="0.425" width="0.05" layer="116"/>
+<circle x="76.835" y="23.812" radius="0.425" width="0.05" layer="116"/>
+<circle x="57.785" y="30.48" radius="0.425" width="0.05" layer="116"/>
+<circle x="36.02" y="29.845" radius="0.425" width="0.05" layer="116"/>
+<circle x="33.02" y="29.845" radius="0.425" width="0.05" layer="116"/>
+<circle x="30.02" y="29.845" radius="0.425" width="0.05" layer="116"/>
+<circle x="30.02" y="23.812" radius="0.425" width="0.05" layer="116"/>
+<circle x="33.02" y="23.812" radius="0.425" width="0.05" layer="116"/>
+<circle x="36.02" y="23.812" radius="0.425" width="0.05" layer="116"/>
+<circle x="90.488" y="29.655" radius="0.425" width="0.05" layer="116"/>
+<circle x="90.488" y="25.591" radius="0.425" width="0.05" layer="116"/>
+<circle x="43.498" y="29.655" radius="0.424" width="0.05" layer="116"/>
+<circle x="43.498" y="25.591" radius="0.424" width="0.05" layer="116"/>
+<circle x="21.908" y="27.94" radius="0.425" width="0.05" layer="116"/>
+<circle x="21.908" y="26.035" radius="0.425" width="0.05" layer="116"/>
+<circle x="52.388" y="25.559" radius="0.424" width="0.05" layer="116"/>
+<circle x="94.933" y="20.955" radius="0.425" width="0.05" layer="116"/>
+<circle x="86.995" y="21.273" radius="0.425" width="0.05" layer="116"/>
+<circle x="77.788" y="38.735" radius="0.425" width="0.05" layer="116"/>
+<circle x="103.188" y="28.258" radius="0.349" width="0.2" layer="116"/>
+<circle x="98.108" y="28.258" radius="0.349" width="0.2" layer="116"/>
+<circle x="116.396" y="23.495" radius="0.35" width="0.2" layer="116"/>
+<circle x="101.41" y="23.495" radius="0.35" width="0.2" layer="116"/>
+<circle x="82.233" y="23.812" radius="0.349" width="0.2" layer="116"/>
+<circle x="82.233" y="26.353" radius="0.349" width="0.2" layer="116"/>
+<circle x="82.233" y="28.893" radius="0.349" width="0.2" layer="116"/>
+<circle x="82.233" y="31.433" radius="0.349" width="0.2" layer="116"/>
+<circle x="76.835" y="31.433" radius="0.35" width="0.2" layer="116"/>
+<circle x="76.835" y="28.893" radius="0.35" width="0.2" layer="116"/>
+<circle x="76.835" y="26.353" radius="0.35" width="0.2" layer="116"/>
+<circle x="76.835" y="23.812" radius="0.35" width="0.2" layer="116"/>
+<circle x="57.785" y="30.48" radius="0.35" width="0.2" layer="116"/>
+<circle x="36.02" y="29.845" radius="0.35" width="0.2" layer="116"/>
+<circle x="33.02" y="29.845" radius="0.35" width="0.2" layer="116"/>
+<circle x="30.02" y="29.845" radius="0.35" width="0.2" layer="116"/>
+<circle x="30.02" y="23.812" radius="0.35" width="0.2" layer="116"/>
+<circle x="33.02" y="23.812" radius="0.35" width="0.2" layer="116"/>
+<circle x="36.02" y="23.812" radius="0.35" width="0.2" layer="116"/>
+<circle x="90.488" y="29.655" radius="0.35" width="0.2" layer="116"/>
+<circle x="90.488" y="25.591" radius="0.35" width="0.2" layer="116"/>
+<circle x="43.498" y="29.655" radius="0.35" width="0.2" layer="116"/>
+<circle x="43.498" y="25.591" radius="0.35" width="0.2" layer="116"/>
+<circle x="98.82" y="4.01" radius="0.325" width="0.15" layer="116"/>
+<circle x="83.82" y="4.01" radius="0.325" width="0.15" layer="116"/>
+<circle x="83.82" y="9.01" radius="0.325" width="0.15" layer="116"/>
+<circle x="83.82" y="14.01" radius="0.325" width="0.15" layer="116"/>
+<circle x="83.82" y="16.51" radius="0.325" width="0.15" layer="116"/>
+<circle x="98.82" y="16.51" radius="0.325" width="0.15" layer="116"/>
+<circle x="83.82" y="11.51" radius="0.325" width="0.15" layer="116"/>
+<circle x="98.82" y="14.01" radius="0.325" width="0.15" layer="116"/>
+<circle x="83.82" y="6.51" radius="0.325" width="0.15" layer="116"/>
+<circle x="21.908" y="27.94" radius="0.35" width="0.2" layer="116"/>
+<circle x="21.908" y="26.035" radius="0.35" width="0.2" layer="116"/>
+<circle x="52.388" y="25.559" radius="0.35" width="0.2" layer="116"/>
+<circle x="94.933" y="20.955" radius="0.349" width="0.2" layer="116"/>
+<circle x="86.995" y="21.273" radius="0.35" width="0.2" layer="116"/>
+<circle x="77.788" y="38.735" radius="0.35" width="0.2" layer="116"/>
 </plain>
 <attributes>
@@
 <wire x1="100.015" y1="42.8625" x2="99.06" y2="42.06625" width="0.8128" layer="1"/>
 </signal>
+<signal name="N$5">
+<wire x1="0" y1="0" x2="0" y2="47.625" width="0.4064" layer="1"/>
+<wire x1="0" y1="47.625" x2="120.3325" y2="47.625" width="0.4064" layer="1"/>
+<wire x1="120.3325" y1="47.625" x2="120.3325" y2="0" width="0.4064" layer="1"/>
+<wire x1="120.3325" y1="0" x2="0" y2="0" width="0.4064" layer="1"/>
+</signal>
 </signals>
