File: Geiger.sch (EAGLE design)
At the start: 35 parts, among them IC1 TINY15LS, IC2 TP4056

Commit message: updates
Parts:
- added C7: (no value), resistor:C-EU225-074X268
- added R10: 50K, resistor:R-EU_R0805
- added R9: 1M, resistor:R-EU_R0805
- SP1, SP2: value AL60P -> AL11P; device buzzer:AL60P -> buzzer:AL11P
Connections:
- removed net N$10: ZD2.A
- removed net TR_PULSE: IC1.(ADC3)PB4, R1.1
- new net VMEASURE: IC1.(ADC3)PB4, R1.1, R10.2, R9.2
- net GND: now also C7.2, R10.1, ZD2.A
- net N$8: now also C7.1
- net VCC: now also R9.1
Other:
- moved on the sheet: C4, D4, R2, R3, R4, R5, R8, SP1, SP2, T2, T3, T4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

Commit message: ahoj
Parts:
- removed S1: TL36PO, switch:TL36PO
- added JP3: PROGRAMMING, pinhead:PINHD-1X4
- added R11: 1M, resistor:R-EU_R0805
- added T5: (no value), transistor:-NPN-SOT23-EBC
- C7: value (none) -> 100n 1KV
Connections:
- removed net N$17: C5.1, IC2.BAT, JP1.1, S1.P
- new net SPKR: SP1.2, T3.C
- net GND: now also JP3.4, T5.E
- net N$14: now also T5.B
- net N$22: now also JP3.3
- net N$23: now also JP3.2
- net PULSE: now also JP3.1, R11.2, T5.C; no longer SP1.2, T3.C
- net VCC: now also C5.1, IC2.BAT, JP1.1, R11.1; no longer S1.O
Other:
- moved on the sheet: JP1, R10, R9

Commit message: dalsi
Parts:
- removed C7: 100n 1KV, resistor:C-EU225-074X268
- removed R6: 0R39, resistor:R-EU_R1206
- removed T2: (no value), transistor:-PNP-SOT23-BCE
- added C8: 100n, resistor:C-EUC0805
- added C9: 100n 500V, resistor:C-EU150-054X183
- added JP4: RESET, pinhead:PINHD-1X1
- added R12: 0R39, resistor:R-EU_R2512
- T1: device transistor:-NPN-SOT23-EBC -> transistor:BC807-16-PNP-SOT23-BEC
- T3, T4, T5: device transistor:-NPN-SOT23-EBC -> transistor:MMBT3904LT1-NPN-SOT23-BEC
Connections:
- removed net N$21: R6.2, U1.VBUS
- new net GNDUSB: R12.2, U1.VBUS
- new net N$10: R11.1, R5.2, T1.C
- net ALARM: now also C8.1, R10.2, R9.2
- net GND: now also C8.2, C9.2; no longer C7.2, T1.E
- net N$12: now also T1.B; no longer T2.B
- net N$13: now also IC1.(ADC0)PB5, JP4.1; no longer R5.2, T2.C
- net N$14: no longer T5.B
- net N$16: now also R12.1; no longer R6.1
- net N$18: now also T5.C; no longer T1.C
- net N$4: now also T5.B; no longer T1.B
- net N$8: now also C9.1; no longer C7.1
- net PULSE: no longer T5.C
- net VCC: now also T1.E; no longer R11.1, T2.E
- net VMEASURE: no longer R10.2, R9.2
Other:
- moved on the sheet: R11, R5, R8, SP1, SP2, T3, T4, T5

Commit message: co asi
Parts:
- removed IC2: TP4056, TP4056:TP4056
- removed JP1: BATTERY, pinhead:PINHD-1X2
- removed R12: 0R39, resistor:R-EU_R2512
- removed U1: (no value), MicroUSB:USB""
- added IC3: TP4056, Geiger:TP4056
- added R6: 1M, resistor:R-EU_0207/7
- added S1: TL36PO, switch:TL36PO
- added U2: USB, Geiger:USB""
- R2: value 1M -> 0R39; device resistor:R-EU_R0805 -> resistor:R-EU_R1206
- R3: value 5M1 -> 4M3
- T1: value (none) -> BC807
- T3, T4, T5: value (none) -> 3904
Connections:
- net N$6 renamed 200V2
- net N$7 renamed 400V3
- net N$9 renamed 200V
- removed net GNDUSB: R12.2, U1.VBUS
- removed net N$5: C4.1, R2.2, R3.1
- removed net N$8: C9.1, D3.C, R2.1, ZD1.C
- new net 400V: C9.1, D3.C, R6.1, ZD1.C
- new net 400V2: C4.1, R3.1, R6.2
- new net N$15: S1.P, S1.S
- new net VCCUSB: R2.2, U2.VBUS
- net GND: now also IC3.GND, IC3.TEMP, IC3.THPAD, JP2.2, U2.GND; no longer IC2.GND, IC2.TEMP, JP1.2, JP2.4, U1.GND
- net N$16: now also IC3.CE, IC3.VCC, R2.1; no longer IC2.CE, IC2.VCC, R12.1
- net N$19: now also IC3.PROG; no longer IC2.PROG
- net N$22: now also JP2.3; no longer JP2.1
- net N$23: now also JP2.4; no longer JP2.2
- net V+: now also JP2.1; no longer JP2.3
- net VCC: now also IC3.BAT, S1.O; no longer IC2.BAT, JP1.1
Other:
- moved on the sheet: R2

Commit message: dalsi
Parts:
- removed D1, D2, D3: BAV21W, diode:MBR0520LT
- added D5, D6, D7: EGL1G, diode:PMLL4150
- added R12, R13, R14: 1M, resistor:R-EU_R0805
- R3: value 4M3 -> 1M
- R6: device resistor:R-EU_0207/7 -> resistor:R-EU_R0805
Connections:
- net VMEASURE renamed OSC
- removed net N$11: R3.2, U$1.P$1
- new net N$6: R3.1, R6.2
- new net N$7: R13.2, R6.1
- new net N$8: R14.1, U$1.P$1
- new net N$9: R13.1, R14.2
- net 200V2: now also D5.C, D6.A; no longer D1.C, D2.A
- net 400V: now also D7.C, R12.1; no longer D3.C, R6.1
- net 400V2: now also R12.2, R3.2; no longer R3.1, R6.2
- net 400V3: now also D6.C, D7.A; no longer D2.C, D3.A
- net GND: now also D5.A; no longer D1.A
Other:
- moved on the sheet: R3, R6
Changed lines of the file:
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@@
 <part name="GND2" library="supply1" deviceset="GND" device=""/>
 <part name="C2" library="resistor" deviceset="C-EU" device="C1206" value="4n7 500V"/>
-<part name="D1" library="diode" deviceset="MBR0520LT" device="" value="BAV21W"/>
 <part name="GND3" library="supply1" deviceset="GND" device=""/>
 <part name="C3" library="resistor" deviceset="C-EU" device="C1206" value="4n7 500V"/>
-<part name="D2" library="diode" deviceset="MBR0520LT" device="" value="BAV21W"/>
-<part name="D3" library="diode" deviceset="MBR0520LT" device="" value="BAV21W"/>
 <part name="ZD1" library="diodes2" deviceset="ZD-" device="MLL-41" value="200V"/>
 <part name="ZD2" library="diodes2" deviceset="ZD-" device="MLL-41" value="200V"/>
 <part name="U$1" library="Geiger" deviceset="SBM-20" device=""/>
-<part name="GND5" library="supply1" deviceset="GND" device=""/>
-<part name="R3" library="resistor" deviceset="R-EU_" device="R0805" value="4M3"/>
 <part name="C4" library="resistor" deviceset="C-EU" device="050-024X044" value="22p 500V"/>
 <part name="R4" library="resistor" deviceset="R-EU_" device="R0805" value="1M"/>
@@
 <part name="IC3" library="Geiger" deviceset="TP4056" device=""/>
 <part name="R2" library="resistor" deviceset="R-EU_" device="R1206" value="0R39"/>
-<part name="R6" library="resistor" deviceset="R-EU_" device="0207/7" value="1M"/>
+<part name="R12" library="resistor" deviceset="R-EU_" device="R0805" value="1M"/>
+<part name="R3" library="resistor" deviceset="R-EU_" device="R0805" value="1M"/>
+<part name="R6" library="resistor" deviceset="R-EU_" device="R0805" value="1M"/>
+<part name="R13" library="resistor" deviceset="R-EU_" device="R0805" value="1M"/>
+<part name="R14" library="resistor" deviceset="R-EU_" device="R0805" value="1M"/>
+<part name="GND5" library="supply1" deviceset="GND" device=""/>
+<part name="D5" library="diode" deviceset="PMLL4150" device="" value="EGL1G"/>
+<part name="D6" library="diode" deviceset="PMLL4150" device="" value="EGL1G"/>
+<part name="D7" library="diode" deviceset="PMLL4150" device="" value="EGL1G"/>
 </parts>
 <sheets>
@@
 <attribute name="VALUE" x="156.464" y="81.661" size="1.778" layer="96"/>
 </instance>
-<instance part="D1" gate="G$1" x="165.1" y="73.66" smashed="yes" rot="R90">
-<attribute name="NAME" x="162.56" y="73.1774" size="1.778" layer="95" rot="R180"/>
-<attribute name="VALUE" x="154.94" y="68.8086" size="1.778" layer="96"/>
-</instance>
 <instance part="GND3" gate="1" x="165.1" y="58.42"/>
 <instance part="C3" gate="G$1" x="170.18" y="68.58" smashed="yes" rot="R90">
@@
 <attribute name="VALUE" x="171.704" y="61.341" size="1.778" layer="96"/>
 </instance>
-<instance part="D2" gate="G$1" x="172.72" y="78.74" smashed="yes">
-<attribute name="NAME" x="170.18" y="84.3026" size="1.778" layer="95"/>
-<attribute name="VALUE" x="170.18" y="81.5086" size="1.778" layer="96"/>
-</instance>
-<instance part="D3" gate="G$1" x="182.88" y="78.74" smashed="yes">
-<attribute name="NAME" x="182.88" y="84.3026" size="1.778" layer="95"/>
-<attribute name="VALUE" x="182.88" y="81.5086" size="1.778" layer="96"/>
-</instance>
 <instance part="ZD1" gate="G$1" x="200.66" y="73.66" rot="R90"/>
 <instance part="ZD2" gate="G$1" x="200.66" y="66.04" rot="R90"/>
-<instance part="U$1" gate="G$1" x="215.9" y="50.8"/>
-<instance part="GND5" gate="1" x="215.9" y="25.4"/>
-<instance part="R3" gate="G$1" x="215.9" y="71.12" rot="R270"/>
+<instance part="U$1" gate="G$1" x="231.14" y="50.8"/>
 <instance part="C4" gate="G$1" x="220.98" y="78.74" rot="R90"/>
 <instance part="R4" gate="G$1" x="231.14" y="86.36" rot="R90"/>
@@
 <instance part="IC3" gate="G$1" x="83.82" y="111.76"/>
 <instance part="R2" gate="G$1" x="86.36" y="127" rot="R90"/>
-<instance part="R6" gate="G$1" x="208.28" y="78.74"/>
+<instance part="R12" gate="G$1" x="208.28" y="78.74"/>
+<instance part="R3" gate="G$1" x="210.82" y="66.04" rot="R90"/>
+<instance part="R6" gate="G$1" x="215.9" y="66.04" rot="R270"/>
+<instance part="R13" gate="G$1" x="220.98" y="66.04" rot="R90"/>
+<instance part="R14" gate="G$1" x="226.06" y="66.04" rot="R270"/>
+<instance part="GND5" gate="1" x="231.14" y="25.4"/>
+<instance part="D5" gate="G$1" x="165.1" y="73.66" rot="R90"/>
+<instance part="D6" gate="G$1" x="172.72" y="78.74"/>
+<instance part="D7" gate="G$1" x="182.88" y="78.74"/>
 </instances>
 <busses>
@@
 </segment>
 <segment>
-<pinref part="D1" gate="G$1" pin="A"/>
 <wire x1="165.1" y1="71.12" x2="165.1" y2="68.58" width="0.1524" layer="91"/>
 <pinref part="GND3" gate="1" pin="GND"/>
@@
 <wire x1="167.64" y1="68.58" x2="165.1" y2="68.58" width="0.1524" layer="91"/>
 <junction x="165.1" y="68.58"/>
+<pinref part="D5" gate="G$1" pin="A"/>
 </segment>
 <segment>
@@
 </segment>
 <segment>
-<pinref part="GND5" gate="1" pin="GND"/>
-<pinref part="U$1" gate="G$1" pin="P$2"/>
-<wire x1="215.9" y1="27.94" x2="215.9" y2="30.48" width="0.1524" layer="91"/>
-</segment>
-<segment>
 <pinref part="GND4" gate="1" pin="GND"/>
 <wire x1="149.86" y1="25.4" x2="149.86" y2="30.48" width="0.1524" layer="91"/>
@@
 <wire x1="157.48" y1="30.48" x2="149.86" y2="30.48" width="0.1524" layer="91"/>
 </segment>
+<segment>
+<pinref part="U$1" gate="G$1" pin="P$2"/>
+<pinref part="GND5" gate="1" pin="GND"/>
+<wire x1="231.14" y1="30.48" x2="231.14" y2="27.94" width="0.1524" layer="91"/>
+</segment>
 </net>
 <net name="N$4" class="0">
@@
 <pinref part="C2" gate="G$1" pin="2"/>
 <wire x1="162.56" y1="78.74" x2="165.1" y2="78.74" width="0.1524" layer="91"/>
-<pinref part="D1" gate="G$1" pin="C"/>
 <wire x1="165.1" y1="76.2" x2="165.1" y2="78.74" width="0.1524" layer="91"/>
-<pinref part="D2" gate="G$1" pin="A"/>
 <wire x1="165.1" y1="78.74" x2="170.18" y2="78.74" width="0.1524" layer="91"/>
 <junction x="165.1" y="78.74"/>
+<pinref part="D5" gate="G$1" pin="C"/>
+<pinref part="D6" gate="G$1" pin="A"/>
 </segment>
 </net>
@@
 <wire x1="175.26" y1="68.58" x2="177.8" y2="68.58" width="0.1524" layer="91"/>
 <wire x1="177.8" y1="68.58" x2="177.8" y2="78.74" width="0.1524" layer="91"/>
-<pinref part="D2" gate="G$1" pin="C"/>
 <wire x1="177.8" y1="78.74" x2="175.26" y2="78.74" width="0.1524" layer="91"/>
-<pinref part="D3" gate="G$1" pin="A"/>
 <wire x1="177.8" y1="78.74" x2="180.34" y2="78.74" width="0.1524" layer="91"/>
 <junction x="177.8" y="78.74"/>
+<pinref part="D6" gate="G$1" pin="C"/>
+<pinref part="D7" gate="G$1" pin="A"/>
 </segment>
 </net>
 <net name="400V" class="0">
 <segment>
-<pinref part="D3" gate="G$1" pin="C"/>
 <pinref part="ZD1" gate="G$1" pin="C"/>
 <wire x1="185.42" y1="78.74" x2="190.5" y2="78.74" width="0.1524" layer="91"/>
@@
 <junction x="190.5" y="78.74"/>
 <pinref part="C9" gate="G$1" pin="1"/>
-<pinref part="R6" gate="G$1" pin="1"/>
+<pinref part="R12" gate="G$1" pin="1"/>
+<pinref part="D7" gate="G$1" pin="C"/>
 </segment>
 </net>
@@
 <net name="400V2" class="0">
 <segment>
-<pinref part="R3" gate="G$1" pin="1"/>
+<pinref part="C4" gate="G$1" pin="1"/>
 <wire x1="213.36" y1="78.74" x2="215.9" y2="78.74" width="0.1524" layer="91"/>
-<pinref part="C4" gate="G$1" pin="1"/>
+<pinref part="R12" gate="G$1" pin="2"/>
+<pinref part="R3" gate="G$1" pin="2"/>
 <wire x1="215.9" y1="78.74" x2="218.44" y2="78.74" width="0.1524" layer="91"/>
-<wire x1="215.9" y1="78.74" x2="215.9" y2="76.2" width="0.1524" layer="91"/>
+<wire x1="210.82" y1="71.12" x2="210.82" y2="76.2" width="0.1524" layer="91"/>
+<wire x1="210.82" y1="76.2" x2="215.9" y2="76.2" width="0.1524" layer="91"/>
+<wire x1="215.9" y1="76.2" x2="215.9" y2="78.74" width="0.1524" layer="91"/>
 <junction x="215.9" y="78.74"/>
-<pinref part="R6" gate="G$1" pin="2"/>
 </segment>
 </net>
@@
 </segment>
 </net>
-<net name="VMEASURE" class="0">
+<net name="OSC" class="0">
 <segment>
 <pinref part="IC1" gate="G$1" pin="(ADC3)PB4"/>
 <pinref part="R1" gate="G$1" pin="1"/>
 <wire x1="101.6" y1="58.42" x2="124.46" y2="58.42" width="0.1524" layer="91"/>
-</segment>
-</net>
-<net name="N$11" class="0">
-<segment>
-<pinref part="U$1" gate="G$1" pin="P$1"/>
-<pinref part="R3" gate="G$1" pin="2"/>
-<wire x1="215.9" y1="63.5" x2="215.9" y2="66.04" width="0.1524" layer="91"/>
 </segment>
 </net>
@@
 </segment>
 </net>
+<net name="N$8" class="0">
+<segment>
+<pinref part="U$1" gate="G$1" pin="P$1"/>
+<wire x1="231.14" y1="73.66" x2="231.14" y2="63.5" width="0.1524" layer="91"/>
+<pinref part="R14" gate="G$1" pin="1"/>
+<wire x1="226.06" y1="71.12" x2="226.06" y2="73.66" width="0.1524" layer="91"/>
+<wire x1="226.06" y1="73.66" x2="231.14" y2="73.66" width="0.1524" layer="91"/>
+</segment>
+</net>
+<net name="N$6" class="0">
+<segment>
+<pinref part="R3" gate="G$1" pin="1"/>
+<wire x1="210.82" y1="60.96" x2="210.82" y2="58.42" width="0.1524" layer="91"/>
+<wire x1="210.82" y1="58.42" x2="215.9" y2="58.42" width="0.1524" layer="91"/>
+<pinref part="R6" gate="G$1" pin="2"/>
+<wire x1="215.9" y1="58.42" x2="215.9" y2="60.96" width="0.1524" layer="91"/>
+</segment>
+</net>
+<net name="N$7" class="0">
+<segment>
+<pinref part="R6" gate="G$1" pin="1"/>
+<wire x1="215.9" y1="71.12" x2="215.9" y2="73.66" width="0.1524" layer="91"/>
+<wire x1="215.9" y1="73.66" x2="220.98" y2="73.66" width="0.1524" layer="91"/>
+<pinref part="R13" gate="G$1" pin="2"/>
+<wire x1="220.98" y1="73.66" x2="220.98" y2="71.12" width="0.1524" layer="91"/>
+</segment>
+</net>
+<net name="N$9" class="0">
+<segment>
+<pinref part="R13" gate="G$1" pin="1"/>
+<wire x1="220.98" y1="60.96" x2="220.98" y2="58.42" width="0.1524" layer="91"/>
+<pinref part="R14" gate="G$1" pin="2"/>
+<wire x1="220.98" y1="58.42" x2="226.06" y2="58.42" width="0.1524" layer="91"/>
+<wire x1="226.06" y1="58.42" x2="226.06" y2="60.96" width="0.1524" layer="91"/>
+</segment>
+</net>
